Commit message: clean mini.xacro and scout_mini.gazebo files

File: src/agilex_scout_sim/scout_description/urdf/mini.xacro (robot description, xacro)
@@ -42,9 +42,4 @@
         </collision>
     </link>
-    <!-- <joint name="chassis_link_joint" type="fixed">
-        <origin xyz="0 0 ${wheel_radius - wheel_vertical_offset}" rpy="0 0 0" />
-        <parent link="base_link" />
-        <child link="chassis_link" />
-    </joint> -->
     <link name="inertial_link">
         <inertial>
